File: schematic/PTBS-1.kicad_sch (KiCad schematic)
At the start: 145 parts, among them J1 MONO PHONE, J15 DC 2.1mm, J2 MONO PHONE, J3 MONO PHONE, J4 MONO PHONE, J5 MONO PHONE, J6 MONO PHONE, J7 MONO PHONE, J8 PHONE STEREO, Q1 2SC1815Y, Q10 2SC1815Y, Q11 2SC1815Y, Q12 2SC1815Y, Q13 2SA1358, Q2 2SC1815Y, Q3 2SC1815, Q4 2SC1815Y, Q5 2SC1815Y, Q6 2SC1815Y, Q7 2SK660, Q8 2SA1015Y, Q9 2SC1815Y, SW1 SW_Push, SW2 SW_Push, SW3 SW_Push, SW4 SW_Push, SW5 SW_Push, SW6 SW_Push, SW7 SW_Push, SW8 SW_Push, U1 L7805, U2 PIC16F873A, U3 SM420561N, X1 10.0MT

Commit message: Add some net names.
Parts:
- U3: value SM420561N -> NAR161H-F
Connections:
- net LED_PGM: now reaches R47.1, U2.14 (RC3/SCK/SCL)
- net CTL: now reaches R48.2, S2.3 (C), U2.12 (RC1/T1OSI/CCP2)
- net LED_MAN: now reaches R46.1, U2.13 (RC2/CCP1)
- net LEDS_ON: now reaches Q9.3 (B), U2.15 (RC4/SDI/SDA)
- net 7SEG_ON: now reaches Q10.3 (B), U2.16 (RC5/SDO)
- net FOOT_SW: now reaches R22.1, R23.2, U2.2 (AN0/RA0)
- net LOOP: now reaches J5.S, J6.S, RY6.11, RY6.8, S2.1 (A)
- net b: now reaches R20.2, U3.6 (B)
Other:
- title: Noa's Ark PTBS-1 -> Noa's Ark PTBS-1 Programmable True Bypass Switcher
- moved on the sheet: LED13, R22, R23, R24, R25, R26, R27, R28, R29, R30, R51, R52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
