File: schematic/PTBS-1.kicad_sch (KiCad schematic)
At the start: 145 parts, among them J1 MONO PHONE, J15 DC 2.1mm, J2 MONO PHONE, J3 MONO PHONE, J4 MONO PHONE, J5 MONO PHONE, J6 MONO PHONE, J7 MONO PHONE, J8 PHONE STEREO, Q1 2SC1815Y, Q10 2SC1815Y, Q11 2SC1815Y, Q12 2SC1815Y, Q13 2SA1358, Q2 2SC1815Y, Q3 2SC1815, Q4 2SC1815Y, Q5 2SC1815Y, Q6 2SC1815Y, Q7 2SK660, Q8 2SA1015Y, Q9 2SC1815Y, SW1 SW_Push, SW2 SW_Push, SW3 SW_Push, SW4 SW_Push, SW5 SW_Push, SW6 SW_Push, SW7 SW_Push, SW8 SW_Push, U1 L7805, U2 PIC16F873A, U3 NAR161H-F, X1 10.0MT

Commit message: I split the schematics into original and modified versions.
Parts:
- removed C1, C2, C5: 0.1u, symbol Device:C
- removed C10: 100p, symbol Device:C
- removed C3, C6: 1u/50V, symbol Device:C_Polarized
- removed C7 (x2): 10u/25V, symbol Device:C_Polarized
- removed C7, C8: 100u/25V, symbol Device:C_Polarized
- removed C7: 470u/16V, symbol Device:C_Polarized
- removed D1, D2, D3, D4, D5, D6, D7, D8: D, symbol Device:D
- removed J1, J2, J3 (x2), J4 (x2), J5 (x3), J6 (x3), J7: MONO PHONE, symbol Connector_Audio:AudioJack2_SwitchT
- removed J15: DC 2.1mm, symbol Connector:Jack-DC
- removed J8: PHONE STEREO, symbol Connector_Audio:AudioJack3
- removed L1, L2: 220u, symbol Device:L_Ferrite
- removed LED1, LED2, LED3, LED4, LED5, LED6: RED 5mm, symbol Device:LED
- removed LED10, LED11, LED12, LED7, LED8, LED9: GREEN 5mm, symbol Device:LED
- removed LED13: BLUE 5mm, symbol Device:LED
- removed Q1, Q10, Q11, Q12, Q2, Q4, Q5, Q6, Q9: 2SC1815Y, Package_TO_SOT_THT:TO-92_Inline, symbol Transistor_BJT:2SC1815
- removed Q13: 2SA1358, Package_TO_SOT_THT:TO-92_Inline, symbol Transistor_BJT:2SA1015
- removed Q3: 2SC1815, Package_TO_SOT_THT:TO-92_Inline, symbol Transistor_BJT:2SC1815
- removed Q7: 2SK660, symbol Simulation_SPICE:NJFET
- removed Q8: 2SA1015Y, Package_TO_SOT_THT:TO-92_Inline, symbol Transistor_BJT:2SA1015
- removed R1, R2, R23, R3, R4, R45, R48, R5, R50, R6 (x2), R8: 10k, symbol Device:R
- removed R10, R11, R12, R13, R14, R15, R20, R58, R9: 470, symbol Device:R
- removed R16, R17, R18, R19, R2, R51, R52, R7: 2k2, symbol Device:R
- removed R21, R31, R32, R33: 220, symbol Device:R
- removed R22, R24, R25, R26, R27, R28, R29, R30, R46, R47: 1k, symbol Device:R
- removed R34, R35, R36, R37, R38, R39, R40, R41, R49, R53, R54, R55, R56: 4M7, symbol Device:R
- removed R43, R57: 2.2k, symbol Device:R
- removed R59: 5k6, symbol Device:R
- removed R60, R61: 4k7, symbol Device:R
- removed R62: 100, symbol Device:R
- removed RY1, RY2, RY3, RY4, RY5, RY6, RY7: G5V-2, Relay_THT:Relay_DPDT_Omron_G5V-2, symbol Relay:G5V-2
- removed S1, S2: SW_DPDT_x2, symbol Switch:SW_DPDT_x2
- removed SW1, SW2, SW3, SW4, SW5, SW6, SW7, SW8: SW_Push, symbol Switch:SW_Push
- removed U1: L7805, symbol Regulator_Linear:L7805
- removed U2: PIC16F873A, symbol MCU_Microchip_PIC16:PIC16F873-XXISP
- removed U3: NAR161H-F, Display_7Segment:7SegmentLED_LTS6760_LTS6780, symbol Display_Character:SM420561N
- removed X1: 10.0MT, symbol Device:Crystal_GND2
Connections:
- no-connect marks 3 -> 0
Other:
- added sheet Modification A (PTBS-1_modA.kicad_sch)
- added sheet Original (PTBS-1_Original.kicad_sch)
